Commit message: add cartesian demo

File: spesbot_description/urdf/arm.xacro (robot description, xacro)
@@ -28,5 +28,5 @@
       <parent link="arm_link_1" />
       <child link="arm_link_2" />
-      <origin xyz="-0.02 0 0.012" rpy="0 0 0" />
+      <origin xyz="0.02 0 0.012" rpy="0 0 0" />
       <axis xyz="0 1 0" />
       <limit lower="-1.57" upper="1.57" effort="100" velocity="0.5" />
@@ -85,4 +85,10 @@
       </visual>
     </link>
+    <joint name="arm_tcp_joint" type="fixed">
+      <parent link="arm_link_5" />
+      <child link="arm_tcp_link" />
+      <origin xyz="0.1 0 0" rpy="0 0 0" />
+    </joint>
+    <link name="arm_tcp_link" />
   </xacro:macro>
 </robot>

File: spesbot_description/urdf/spesbot.xacro (robot description, xacro)
@@ -10,3 +10,36 @@
         <origin xyz="0 0.08 0.08" rpy="0 0 0" />
     </joint>
+    <ros2_control name="fake_system" type="system">
+        <hardware>
+            <plugin>mock_components/GenericSystem</plugin>
+        </hardware>
+        <joint name="joint_1">
+            <command_interface name="position" />
+            <state_interface name="position" />
+        </joint>
+        <joint name="joint_2">
+            <command_interface name="position" />
+            <state_interface name="position" />
+        </joint>
+        <joint name="joint_3">
+            <command_interface name="position" />
+            <state_interface name="position" />
+        </joint>
+        <joint name="joint_4">
+            <command_interface name="position" />
+            <state_interface name="position" />
+        </joint>
+        <joint name="joint_5">
+            <command_interface name="position" />
+            <state_interface name="position" />
+        </joint>
+        <joint name="left_motor">
+            <command_interface name="velocity" />
+            <state_interface name="position" />
+        </joint>
+        <joint name="right_motor">
+            <command_interface name="velocity" />
+            <state_interface name="position" />
+        </joint>
+    </ros2_control>
 </robot>
