Commit message: merge models

File: spesbot_description/urdf/mobile_base.xacro (robot description, xacro)
@@ -13,6 +13,6 @@
             <parent link="base_link" />
             <child link="left_wheel_link" />
-            <origin xyz="0 0.1 0" rpy="0 0 0" />
-            <axis xyz="0 0 1" />
+            <origin xyz="0 0.145 0" rpy="0 0 0" />
+            <axis xyz="0 1 0" />
         </joint>
         <link name="left_wheel_link">
@@ -20,5 +20,48 @@
                 <geometry>
                     <mesh
-                        filename="package://spesbot_description/urdf/meshes/simplified/wheel.stl" />
+                        filename="package://spesbot_description/urdf/meshes/wheel.stl" />
+                </geometry>
+            </visual>
+        </link>
+        <joint name="right_motor" type="continuous">
+            <parent link="base_link" />
+            <child link="right_wheel_link" />
+            <origin xyz="0 -0.145 0" rpy="0 0 0" />
+            <axis xyz="0 1 0" />
+        </joint>
+        <link name="right_wheel_link">
+            <visual>
+                <geometry>
+                    <mesh
+                        filename="package://spesbot_description/urdf/meshes/wheel.stl" />
+                </geometry>
+                <origin xyz="0 0 0" rpy="0 0 3.14159" />
+            </visual>
+        </link>
+        <joint name="caster_steering_joint" type="continuous">
+            <parent link="base_link" />
+            <child link="caster_holder_link" />
+            <origin xyz="-0.31 0 0" rpy="0 0 0" />
+            <axis xyz="0 0 1" />
+        </joint>
+        <link name="caster_holder_link">
+            <visual>
+                <geometry>
+                    <mesh
+                        filename="package://spesbot_description/urdf/meshes/caster_holder.stl" />
+                </geometry>
+            </visual>
+        </link>
+        <joint name="caster_wheel_joint" type="continuous">
+            <parent link="caster_holder_link" />
+            <child link="caster_wheel_link" />
+            <origin xyz="-0.03 0 -0.05" rpy="0 0 0" />
+            <axis xyz="0 1 0" />
+        </joint>
+        <link name="caster_wheel_link">
+            <visual>
+                <geometry>
+                    <mesh
+                        filename="package://spesbot_description/urdf/meshes/caster_wheel.stl" />
                 </geometry>
             </visual>

File: spesbot_description/urdf/spesbot.xacro (robot description, xacro)
@@ -2,8 +2,11 @@
 <robot name="spesbot" xmlns:xacro="http://ros.org/wiki/xacro">
     <xacro:include filename="$(find spesbot_description)/urdf/mobile_base.xacro" />
-    <!-- <xacro:include filename="$(find spesbot_description)/urdf/spesbot_arm.xacro" /> -->
+    <xacro:include filename="$(find spesbot_description)/urdf/arm.xacro" />
     <xacro:mobile_base />
-    <!-- <xacro:arm parent="base_link">
-        <origin xyz="0.1 0 0.1" rpy="0 0 0" />
-    </xacro:arm> -->
+    <xacro:arm />
+    <joint name="arm_fixed_joint" type="fixed">
+        <parent link="base_link" />
+        <child link="arm_base_link" />
+        <origin xyz="0 0.08 0.08" rpy="0 0 0" />
+    </joint>
 </robot>

Commit message: Use mesh in the Webots model

File: spesbot_description/urdf/mobile_base.xacro (robot description, xacro)
@@ -9,4 +9,15 @@
                 </geometry>
             </visual>
+            <collision>
+                <geometry>
+                    <origin xyz="-0.15 0 0" rpy="0 0 0" />
+                    <box size="0.4 0.3 0.02" />
+                </geometry>
+            </collision>
+            <inertial>
+                <mass value="5.0" />
+                <origin xyz="0 0 0" rpy="0 0 0" />
+                <inertia ixx="0.1" ixy="0" ixz="0" iyy="0.1" iyz="0" izz="0.1" />
+            </inertial>
         </link>
         <joint name="left_motor" type="continuous">
@@ -23,4 +34,15 @@
                 </geometry>
             </visual>
+            <collision>
+                <origin xyz="0 0.03 0" rpy="1.5707 0 0" />
+                <geometry>
+                    <cylinder radius="0.085" length="0.03"/>
+                </geometry>
+            </collision>
+            <inertial>
+                <mass value="2.0" />
+                <origin xyz="0 0 0" rpy="0 0 0" />
+                <inertia ixx="0.0001" ixy="0" ixz="0" iyy="0.0001" iyz="0" izz="0.0001" />
+            </inertial>
         </link>
         <joint name="right_motor" type="continuous">
@@ -38,4 +60,15 @@
                 <origin xyz="0 0 0" rpy="0 0 3.14159" />
             </visual>
+            <collision>
+                <origin xyz="0 -0.03 0" rpy="1.5707 0 0" />
+                <geometry>
+                    <cylinder radius="0.085" length="0.03"/>
+                </geometry>
+            </collision>
+            <inertial>
+                <mass value="2.0" />
+                <origin xyz="0 0 0" rpy="0 0 0" />
+                <inertia ixx="0.0001" ixy="0" ixz="0" iyy="0.0001" iyz="0" izz="0.0001" />
+            </inertial>
         </link>
         <joint name="caster_steering_joint" type="continuous">
@@ -52,4 +85,15 @@
                 </geometry>
             </visual>
+            <collision>
+                <origin xyz="0 0 0" rpy="0 0 0" />
+                <geometry>
+                    <cylinder radius="0.03" length="0.01"/>
+                </geometry>
+            </collision>
+            <inertial>
+                <mass value="0.3" />
+                <origin xyz="0 0 0" rpy="0 0 0" />
+                <inertia ixx="0.0001" ixy="0" ixz="0" iyy="0.0001" iyz="0" izz="0.0001" />
+            </inertial>
         </link>
         <joint name="caster_wheel_joint" type="continuous">
@@ -66,5 +110,19 @@
                 </geometry>
             </visual>
+            <collision>
+                <origin xyz="0 0 0" rpy="1.5707 0 0" />
+                <geometry>
+                    <cylinder radius="0.033" length="0.03"/>
+                </geometry>
+            </collision>
+            <inertial>
+                <mass value="2.0" />
+                <origin xyz="0 0 0" rpy="0 0 0" />
+                <inertia ixx="0.0001" ixy="0" ixz="0" iyy="0.0001" iyz="0" izz="0.0001" />
+            </inertial>
         </link>
+        <gazebo reference="caster_wheel_link">
+            <material>Gazebo/Black</material>
+          </gazebo>
     </xacro:macro>
 </robot>

Commit message: Implementing ros2_control feature for controlling the spesbot in IsaacSim

File: spesbot_description/urdf/mobile_base.xacro (robot description, xacro)
@@ -5,8 +5,18 @@
             <visual>
                 <geometry>
-                    <mesh
-                        filename="package://spesbot_description/urdf/meshes/mobile_base.stl" />
+                    <mesh filename="package://spesbot_description/urdf/meshes/mobile_base.stl"/>
                 </geometry>
             </visual>
+            <collision>
+                <origin xyz="-0.15 0 0" rpy="0 0 0" />
+                <geometry>
+                    <box size="0.4 0.3 0.02" />
+                </geometry>
+            </collision>
+            <inertial>
+                <mass value="5.0" />
+                <origin xyz="0 0 0" rpy="0 0 0" />
+                <inertia ixx="0.1" ixy="0" ixz="0" iyy="0.1" iyz="0" izz="0.1" />
+            </inertial>
         </link>
         <joint name="left_motor" type="continuous">
@@ -19,8 +29,18 @@
             <visual>
                 <geometry>
-                    <mesh
-                        filename="package://spesbot_description/urdf/meshes/wheel.stl" />
+                    <mesh filename="package://spesbot_description/urdf/meshes/wheel.stl"/>
                 </geometry>
             </visual>
+            <collision>
+                <origin xyz="0 0.03 0" rpy="1.5707 0 0" />
+                <geometry>
+                    <cylinder radius="0.085" length="0.03"/>
+                </geometry>
+            </collision>
+            <inertial>
+                <mass value="2.0" />
+                <origin xyz="0 0 0" rpy="0 0 0" />
+                <inertia ixx="0.0001" ixy="0" ixz="0" iyy="0.0001" iyz="0" izz="0.0001" />
+            </inertial>
         </link>
         <joint name="right_motor" type="continuous">
@@ -38,4 +58,15 @@
                 <origin xyz="0 0 0" rpy="0 0 3.14159" />
             </visual>
+            <collision>
+                <origin xyz="0 -0.03 0" rpy="1.5707 0 0" />
+                <geometry>
+                    <cylinder radius="0.085" length="0.03"/>
+                </geometry>
+            </collision>
+            <inertial>
+                <mass value="2.0" />
+                <origin xyz="0 0 0" rpy="0 0 0" />
+                <inertia ixx="0.0001" ixy="0" ixz="0" iyy="0.0001" iyz="0" izz="0.0001" />
+            </inertial>
         </link>
         <joint name="caster_steering_joint" type="continuous">
@@ -52,4 +83,15 @@
                 </geometry>
             </visual>
+            <collision>
+                <origin xyz="0 0 0" rpy="0 0 0" />
+                <geometry>
+                    <cylinder radius="0.03" length="0.01"/>
+                </geometry>
+            </collision>
+            <inertial>
+                <mass value="0.3" />
+                <origin xyz="0 0 0" rpy="0 0 0" />
+                <inertia ixx="0.0001" ixy="0" ixz="0" iyy="0.0001" iyz="0" izz="0.0001" />
+            </inertial>
         </link>
         <joint name="caster_wheel_joint" type="continuous">
@@ -66,4 +108,15 @@
                 </geometry>
             </visual>
+            <collision>
+                <origin xyz="0 0 0" rpy="1.5707 0 0" />
+                <geometry>
+                    <cylinder radius="0.033" length="0.03"/>
+                </geometry>
+            </collision>
+            <inertial>
+                <mass value="2.0" />
+                <origin xyz="0 0 0" rpy="0 0 0" />
+                <inertia ixx="0.0001" ixy="0" ixz="0" iyy="0.0001" iyz="0" izz="0.0001" />
+            </inertial>
         </link>
     </xacro:macro>

File: spesbot_description/urdf/spesbot.xacro (robot description, xacro)
@@ -34,4 +34,12 @@
             <state_interface name="position" />
         </joint>
+    </ros2_control>
+    <ros2_control name="isaac_system" type="system">
+        <hardware>
+            <plugin>topic_based_ros2_control/TopicBasedSystem</plugin>
+            <param name="joint_commands_topic">/joint_command</param>
+            <param name="joint_states_topic">/joint_states</param>
+            <param name="sum_wrapped_joint_states">true</param>
+        </hardware>
         <joint name="left_motor">
             <command_interface name="velocity" />

Commit message: Add .usd and .usda files, rename the .yaml file, format files, rename the topics of topic based hardware interface

File: spesbot_description/urdf/mobile_base.xacro (robot description, xacro)
@@ -5,5 +5,5 @@
             <visual>
                 <geometry>
-                    <mesh filename="package://spesbot_description/urdf/meshes/mobile_base.stl"/>
+                    <mesh filename="package://spesbot_description/urdf/meshes/mobile_base.stl" />
                 </geometry>
             </visual>
@@ -29,5 +29,5 @@
             <visual>
                 <geometry>
-                    <mesh filename="package://spesbot_description/urdf/meshes/wheel.stl"/>
+                    <mesh filename="package://spesbot_description/urdf/meshes/wheel.stl" />
                 </geometry>
             </visual>
@@ -35,5 +35,5 @@
                 <origin xyz="0 0.03 0" rpy="1.5707 0 0" />
                 <geometry>
-                    <cylinder radius="0.085" length="0.03"/>
+                    <cylinder radius="0.085" length="0.03" />
                 </geometry>
             </collision>
@@ -61,5 +61,5 @@
                 <origin xyz="0 -0.03 0" rpy="1.5707 0 0" />
                 <geometry>
-                    <cylinder radius="0.085" length="0.03"/>
+                    <cylinder radius="0.085" length="0.03" />
                 </geometry>
             </collision>
@@ -86,5 +86,5 @@
                 <origin xyz="0 0 0" rpy="0 0 0" />
                 <geometry>
-                    <cylinder radius="0.03" length="0.01"/>
+                    <cylinder radius="0.03" length="0.01" />
                 </geometry>
             </collision>
@@ -111,5 +111,5 @@
                 <origin xyz="0 0 0" rpy="1.5707 0 0" />
                 <geometry>
-                    <cylinder radius="0.033" length="0.03"/>
+                    <cylinder radius="0.033" length="0.03" />
                 </geometry>
             </collision>

File: spesbot_description/urdf/spesbot.xacro (robot description, xacro)
@@ -38,6 +38,6 @@
         <hardware>
             <plugin>topic_based_ros2_control/TopicBasedSystem</plugin>
-            <param name="joint_commands_topic">/joint_command</param>
-            <param name="joint_states_topic">/joint_states</param>
+            <param name="joint_commands_topic">/isaac/joint_command</param>
+            <param name="joint_states_topic">/isaac/joint_states</param>
             <param name="sum_wrapped_joint_states">true</param>
         </hardware>

Commit message: Add feature navsatfix for IsaacSim (#27)
* Adding the feature of ros2_control for the spesbot to IsaacSIm

* Add .usd and .usda files, rename the .yaml file, format files, rename the topics of topic based hardware interface

* navsatfix scripts, yaml file name

* ros2_numpy dependencies and pymap3d

File: spesbot_description/urdf/mobile_base.xacro (robot description, xacro)
@@ -5,8 +5,18 @@
             <visual>
                 <geometry>
-                    <mesh
-                        filename="package://spesbot_description/urdf/meshes/mobile_base.stl" />
+                    <mesh filename="package://spesbot_description/urdf/meshes/mobile_base.stl" />
                 </geometry>
             </visual>
+            <collision>
+                <origin xyz="-0.15 0 0" rpy="0 0 0" />
+                <geometry>
+                    <box size="0.4 0.3 0.02" />
+                </geometry>
+            </collision>
+            <inertial>
+                <mass value="5.0" />
+                <origin xyz="0 0 0" rpy="0 0 0" />
+                <inertia ixx="0.1" ixy="0" ixz="0" iyy="0.1" iyz="0" izz="0.1" />
+            </inertial>
         </link>
         <joint name="left_motor" type="continuous">
@@ -19,8 +29,18 @@
             <visual>
                 <geometry>
-                    <mesh
-                        filename="package://spesbot_description/urdf/meshes/wheel.stl" />
+                    <mesh filename="package://spesbot_description/urdf/meshes/wheel.stl" />
                 </geometry>
             </visual>
+            <collision>
+                <origin xyz="0 0.03 0" rpy="1.5707 0 0" />
+                <geometry>
+                    <cylinder radius="0.085" length="0.03" />
+                </geometry>
+            </collision>
+            <inertial>
+                <mass value="2.0" />
+                <origin xyz="0 0 0" rpy="0 0 0" />
+                <inertia ixx="0.0001" ixy="0" ixz="0" iyy="0.0001" iyz="0" izz="0.0001" />
+            </inertial>
         </link>
         <joint name="right_motor" type="continuous">
@@ -38,4 +58,15 @@
                 <origin xyz="0 0 0" rpy="0 0 3.14159" />
             </visual>
+            <collision>
+                <origin xyz="0 -0.03 0" rpy="1.5707 0 0" />
+                <geometry>
+                    <cylinder radius="0.085" length="0.03" />
+                </geometry>
+            </collision>
+            <inertial>
+                <mass value="2.0" />
+                <origin xyz="0 0 0" rpy="0 0 0" />
+                <inertia ixx="0.0001" ixy="0" ixz="0" iyy="0.0001" iyz="0" izz="0.0001" />
+            </inertial>
         </link>
         <joint name="caster_steering_joint" type="continuous">
@@ -52,4 +83,15 @@
                 </geometry>
             </visual>
+            <collision>
+                <origin xyz="0 0 0" rpy="0 0 0" />
+                <geometry>
+                    <cylinder radius="0.03" length="0.01" />
+                </geometry>
+            </collision>
+            <inertial>
+                <mass value="0.3" />
+                <origin xyz="0 0 0" rpy="0 0 0" />
+                <inertia ixx="0.0001" ixy="0" ixz="0" iyy="0.0001" iyz="0" izz="0.0001" />
+            </inertial>
         </link>
         <joint name="caster_wheel_joint" type="continuous">
@@ -66,4 +108,15 @@
                 </geometry>
             </visual>
+            <collision>
+                <origin xyz="0 0 0" rpy="1.5707 0 0" />
+                <geometry>
+                    <cylinder radius="0.033" length="0.03" />
+                </geometry>
+            </collision>
+            <inertial>
+                <mass value="2.0" />
+                <origin xyz="0 0 0" rpy="0 0 0" />
+                <inertia ixx="0.0001" ixy="0" ixz="0" iyy="0.0001" iyz="0" izz="0.0001" />
+            </inertial>
         </link>
     </xacro:macro>

File: spesbot_description/urdf/spesbot.xacro (robot description, xacro)
@@ -34,4 +34,12 @@
             <state_interface name="position" />
         </joint>
+    </ros2_control>
+    <ros2_control name="isaac_system" type="system">
+        <hardware>
+            <plugin>topic_based_ros2_control/TopicBasedSystem</plugin>
+            <param name="joint_commands_topic">/isaac/joint_command</param>
+            <param name="joint_states_topic">/isaac/joint_states</param>
+            <param name="sum_wrapped_joint_states">true</param>
+        </hardware>
         <joint name="left_motor">
             <command_interface name="velocity" />
