Commit message: add gripper

File: xarm_bringup/urdf/lite6.ros2_control.xacro (robot description, xacro)
@@ -1,5 +1,6 @@
 <?xml version="1.0"?>
 <robot xmlns:xacro="http://ros.org/wiki/xacro">
-  <xacro:macro name="lite6_ros2_control" params="prefix
+  <xacro:macro name="lite6_ros2_control"
+    params="prefix
     velocity_control:='false'
     ros2_control_plugin:='uf_robot_hardware/UFRobotSystemHardware'
@@ -35,6 +36,6 @@
           <param name="max">3.14</param>
         </command_interface>
-        <state_interface name="position"/>
-        <state_interface name="velocity"/>
+        <state_interface name="position" />
+        <state_interface name="velocity" />
         <!-- <state_interface name="effort"/> -->
       </joint>
@@ -48,6 +49,6 @@
           <param name="max">3.14</param>
         </command_interface>
-        <state_interface name="position"/>
-        <state_interface name="velocity"/>
+        <state_interface name="position" />
+        <state_interface name="velocity" />
         <!-- <state_interface name="effort"/> -->
       </joint>
@@ -61,6 +62,6 @@
           <param name="max">3.14</param>
         </command_interface>
-        <state_interface name="position"/>
-        <state_interface name="velocity"/>
+        <state_interface name="position" />
+        <state_interface name="velocity" />
         <!-- <state_interface name="effort"/> -->
       </joint>
@@ -74,6 +75,6 @@
           <param name="max">3.14</param>
         </command_interface>
-        <state_interface name="position"/>
-        <state_interface name="velocity"/>
+        <state_interface name="position" />
+        <state_interface name="velocity" />
         <!-- <state_interface name="effort"/> -->
       </joint>
@@ -87,6 +88,6 @@
           <param name="max">3.14</param>
         </command_interface>
-        <state_interface name="position"/>
-        <state_interface name="velocity"/>
+        <state_interface name="position" />
+        <state_interface name="velocity" />
         <!-- <state_interface name="effort"/> -->
       </joint>
@@ -100,9 +101,22 @@
           <param name="max">3.14</param>
         </command_interface>
-        <state_interface name="position"/>
-        <state_interface name="velocity"/>
+        <state_interface name="position" />
+        <state_interface name="velocity" />
         <!-- <state_interface name="effort"/> -->
       </joint>
     </ros2_control>
   </xacro:macro>
+  <ros2_control name="GripperSystem" type="system">
+    <hardware>
+      <plugin>fake_components/GenericSystem</plugin>
+    </hardware>
+    <joint name="gripper_left_joint">
+      <command_interface name="position" />
+      <state_interface name="position" />
+    </joint>
+    <joint name="gripper_right_joint">
+      <command_interface name="position" />
+      <state_interface name="position" />
+    </joint>
+  </ros2_control>
 </robot>

File: xarm_bringup/urdf/lite6.urdf.xacro (robot description, xacro)
@@ -5,5 +5,5 @@
   <xacro:arg name="limited" default="false" />
   <xacro:arg name="velocity_control" default="false" />
-  <xacro:arg name="add_gripper" default="false" />
+  <xacro:arg name="add_gripper" default="true" />
   <xacro:arg name="robot_ip" default="" />
   <xacro:arg name="report_type" default="normal" />
@@ -14,17 +14,25 @@
   <xacro:arg name="hard_interface" default="PositionJointInterface" />
   <xacro:arg name="inertial_params_filename" default="" />
-  <xacro:arg name="kinematics_params_filename" default="$(find xarm_description)/config/kinematics/default/lite6_default_kinematics.yaml" />
+  <xacro:arg name="kinematics_params_filename"
+    default="$(find xarm_description)/config/kinematics/default/lite6_default_kinematics.yaml" />
   <xacro:arg name="is_ros2" default="true" />
   <xacro:include filename="$(find xarm_description)/urdf/common/common.material.xacro" />
   <xacro:common_material prefix="$(arg prefix)" />
-  <xacro:property name="use_xacro_load_yaml" value="true" scope="global"/>
-  <xacro:property name="mesh_path" value="package://xarm_description/meshes" scope="global"/>
-  <xacro:property name="mesh_suffix" value="stl" scope="global"/>
+  <xacro:property name="use_xacro_load_yaml" value="true" scope="global" />
+  <xacro:property name="mesh_path" value="package://xarm_description/meshes" scope="global" />
+  <xacro:property name="mesh_suffix" value="stl" scope="global" />
   <xacro:include filename="$(find xarm_description)/urdf/common/common.link.xacro" />
   <xacro:if value="$(arg is_ros2)">
     <xacro:include filename="$(find xarm_bringup)/urdf/lite6.ros2_control.xacro" />
   </xacro:if>
+  <xacro:include filename="$(find xarm_bringup)/urdf/lite6_gripper.xacro" />
   <xacro:include filename="$(find xarm_description)/urdf/lite6/lite6.urdf.xacro" />
   <xacro:include filename="$(find xarm_description)/urdf/lite6/lite6.transmission.xacro" />
+  <link name="base_link" />
+  <joint name="base_link_fix_joint" type="fixed">
+    <parent link="base_link" />
+    <child link="link_base" />
+    <origin xyz="0 0 0" rpy="0 0 0" />
+  </joint>
   <xacro:if value="$(arg limited)">
     <xacro:if value="$(arg is_ros2)">
@@ -67,3 +75,11 @@
   </xacro:unless>
   <xacro:lite6_transmission prefix="$(arg prefix)" hard_interface="$(arg hard_interface)" />
+  <xacro:if value="$(arg add_gripper)">
+    <xacro:lite6_gripper />
+    <joint name="gripper_joint" type="fixed">
+      <parent link="link6" />
+      <child link="gripper_base_link" />
+      <origin xyz="0 0 0" rpy="0 0 0" />
+    </joint>
+  </xacro:if>
 </robot>

Commit message: add position controller

File: xarm_bringup/urdf/lite6.ros2_control.xacro (robot description, xacro)
@@ -107,18 +107,9 @@
         <!-- <state_interface name="effort"/> -->
       </joint>
+      <joint name="gripper_left_joint">
+        <command_interface name="position" />
+        <state_interface name="position" />
+      </joint>
     </ros2_control>
   </xacro:macro>
-  <ros2_control name="GripperSystem" type="system">
-    <hardware>
-      <plugin>fake_components/GenericSystem</plugin>
-    </hardware>
-    <joint name="gripper_left_joint">
-      <command_interface name="position" />
-      <state_interface name="position" />
-    </joint>
-    <joint name="gripper_right_joint">
-      <command_interface name="position" />
-      <state_interface name="position" />
-    </joint>
-  </ros2_control>
 </robot>
