Commit message: make custom coliders for gripper

File: xarm_bringup/urdf/lite6_gripper.xacro (robot description, xacro)
@@ -27,5 +27,6 @@
             <collision>
                 <geometry>
-                    <mesh filename="package://xarm_bringup/urdf/meshes/lite6/gripper_finger.stl" />
+                    <!-- <mesh filename="package://xarm_bringup/urdf/meshes/lite6/gripper_finger.stl" /> -->
+                    <box size="0.018 0.018 0.021" />
                 </geometry>
                 <origin rpy="0 0 3.14159" xyz="0 0 0" />
@@ -50,5 +51,6 @@
             <collision>
                 <geometry>
-                    <mesh filename="package://xarm_bringup/urdf/meshes/lite6/gripper_finger.stl" />
+                    <!-- <mesh filename="package://xarm_bringup/urdf/meshes/lite6/gripper_finger.stl" /> -->
+                    <box size="0.018 0.018 0.021" />
                 </geometry>
             </collision>

Commit message: add primitive collisions

File: xarm_bringup/urdf/lite6_gripper.xacro (robot description, xacro)
@@ -10,9 +10,11 @@
             <collision>
                 <geometry>
-                    <mesh filename="package://xarm_bringup/urdf/meshes/lite6/gripper_base.stl" />
+                    <!-- <mesh filename="package://xarm_bringup/urdf/meshes/lite6/gripper_base.stl" /> -->
+                    <cylinder radius="0.035" length="0.05"/>
                 </geometry>
+                <origin rpy="0 0 0" xyz="0 0 0.03" />
             </collision>
             <inertial>
-                <mass value="0.5" />
+                <mass value="0.3" />
                 <inertia ixx="0.02" ixy="0.0" ixz="0.0" iyy="0.02" iyz="0.0" izz="0.01" />
             </inertial>
@@ -28,7 +30,7 @@
                 <geometry>
                     <!-- <mesh filename="package://xarm_bringup/urdf/meshes/lite6/gripper_finger.stl" /> -->
-                    <box size="0.018 0.018 0.021" />
+                    <box size="0.02 0.004 0.021" />
                 </geometry>
-                <origin rpy="0 0 3.14159" xyz="0 0 0" />
+                <origin rpy="0 0 0" xyz="0 -0.022 0.073" />
             </collision>
             <inertial>
@@ -52,6 +54,7 @@
                 <geometry>
                     <!-- <mesh filename="package://xarm_bringup/urdf/meshes/lite6/gripper_finger.stl" /> -->
-                    <box size="0.018 0.018 0.021" />
+                    <box size="0.02 0.004 0.021" />
                 </geometry>
+                <origin rpy="0 0 0" xyz="0 0.022 0.073" />
             </collision>
             <inertial>
